Commit message: Added realsense cameras

File: universal_robot/ur_description/urdf/ur5_joint_limited_robot.urdf.xacro (robot description, xacro)
@@ -17,4 +17,12 @@
     transmission_hw_interface="$(arg transmission_hw_interface)"
   />
+  <!-- Realsense Camera -->
+  <xacro:include filename="$(find ur5_control)/urdf/_d435.urdf.xacro" />
+  <xacro:sensor_d435 parent="world" name="camera_1" topics_ns="camera_1">
+    <origin xyz="1.25 0 0.6" rpy="0 ${pi/12} ${pi}"/>
+  </xacro:sensor_d435>
+  <xacro:sensor_d435 parent="world" name="camera_2" topics_ns="camera_2">
+    <origin xyz="-1.25 0 0.6" rpy="0 ${pi/12} 0.0"/>
+  </xacro:sensor_d435>
   <link name="world" />
   <link name="pedestal">

File: ur5_control/urdf/_d435.gazebo.xacro (robot description, xacro)
@@ -134,9 +134,9 @@
         <infrared2OpticalframeName>${infrared2_optical_frame}</infrared2OpticalframeName>
         <rangeMinDepth>0.2</rangeMinDepth>
-        <rangeMaxDepth>10.0</rangeMaxDepth>
+        <rangeMaxDepth>3.0</rangeMaxDepth>
         <pointCloud>${publish_pointcloud}</pointCloud>
         <pointCloudTopicName>depth/color/points</pointCloudTopicName>
         <pointCloudCutoff>0.25</pointCloudCutoff>
-        <pointCloudCutoffMax>9.0</pointCloudCutoffMax>
+        <pointCloudCutoffMax>3.0</pointCloudCutoffMax>
       </plugin>
     </gazebo>

File: ur5_control/urdf/_d435.urdf.xacro (robot description, xacro)
@@ -8,5 +8,5 @@
 <robot name="sensor_d435" xmlns:xacro="http://ros.org/wiki/xacro">
   <!--File includes-->
-  <xacro:include filename="$(find mmt_ur5e)/urdf/_d435.gazebo.xacro"/>
+  <xacro:include filename="$(find ur5_control)/urdf/_d435.gazebo.xacro"/>
   <xacro:macro name="sensor_d435" params="name:=camera topics_ns:=camera parent *origin publish_pointcloud:=true">
     <xacro:property name="M_PI" value="3.1415926535897931" />
